File: DC34-Mech-SAO/DC34-Mech-SAO.kicad_sch (KiCad schematic)
At the start: 20 parts, among them J1 Conn_01x06_Male, J2 Conn_01x03_Male, U1 ATtiny816-M

Commit message: Updates to project over last few days.
Parts:
- removed J2: Conn_01x03_Male, Connector_PinSocket_2.54mm:PinSocket_1x03_P2.54mm_Vertical, symbol Connector:Conn_01x03_Male
- added J2: Conn_01x01_Male, UPDI_ICRP:Aligator_TIP, symbol Connector:Conn_01x01_Male
- J1: footprint Connector_PinHeader_2.54mm:PinHeader_2x03_P2.54mm_Vertical -> Connector_PinSocket_2.54mm:PinSocket_2x03_P2.54mm_Vertical_SMD
- R1: value 10k -> 2k
Connections:
- net UPDI: now also J2.1 (Pin_1)
